File: KiCAD_prj/ForKids/ArduinoDevBoard/2_0/KiCAD/ArduinoDevBoard_2_0/ArduinoDevBoard_2_0.sch (KiCad schematic (older format))
At the start: 39 parts, among them J1 Conn_01x04_Female, J10 Conn_01x04_Female, J11 Conn_01x04_Female, J12 Conn_01x02_Female, J2 Conn_01x04_Female, J3 Conn_01x05_Female, J4 Screw_Terminal_01x02, J5 Conn_01x02_Female, J6 Conn_01x02_Female, J7 Conn_01x04_Female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

Commit message: Update ArduinoDevBoard 2.0 in KiCad
Parts:
- added C1: 47uF, symbol Device:CP
- added C2: 10uF, symbol Device:CP
- added D7: 1N4007, symbol Device:D
- D6: value D -> 1N4007
- J1, J10, J11, J2, J7: footprint (none) -> Connector_PinHeader_2.54mm:PinHeader_1x04_P2.54mm_Vertical
- J3: footprint (none) -> Connector_PinHeader_2.54mm:PinHeader_1x05_P2.54mm_Vertical
- J4, J8: footprint (none) -> Connector_Phoenix_MC:PhoenixContact_MCV_1,5_2-G-3.5_1x02_P3.50mm_Vertical
- J5, J6, SW1, SW2, SW3: footprint (none) -> Connector_PinHeader_2.54mm:PinHeader_1x02_P2.54mm_Vertical
- J9: footprint (none) -> Connector_PinHeader_2.54mm:PinHeader_1x03_P2.54mm_Vertical
Connections:
- net +12V: now also J5.1 (Pin_1)
- net Earth: now also C1.2, C2.2; no longer J5.1 (Pin_1)
- net at J5.2 (Pin_2), U1.1 (VI): now also C1.1, D7.1 (K)
- net at J6.1 (Pin_1), U1.3 (VO): now also C2.1, D7.2 (A)
Other:
- note added: "Arduino Dev Board 2.1"
- note added: "RGB светодиод"
- note removed: "Arduino Dev Board 2.0"
- moved on the sheet: J7

Commit message: Update ArduinoDevBoard 2.1
Parts:
- added J13, J14: Conn_01x15_Female, symbol Connector:Conn_01x15_Female
- C1, C2: footprint (none) -> Capacitor_THT:CP_Radial_D5.0mm_P2.50mm
- D1, D2, D3, D4, D5: footprint (none) -> LED_THT:LED_D5.0mm
- D6, D7: footprint (none) -> Diode_THT:D_A-405_P7.62mm_Horizontal
- J12: footprint (none) -> Connector_PinHeader_2.54mm:PinHeader_1x02_P2.54mm_Vertical
- Q1: footprint Package_TO_SOT_THT:TO-92_Inline -> Package_TO_SOT_THT:TO-92_Inline_Wide
- R1, R2, R3, R4, R5, R6, R7, R8: footprint (none) -> Resistor_THT:R_Axial_DIN0411_L9.9mm_D3.6mm_P12.70mm_Horizontal
- R10, R11, R9: value R -> 10K; footprint (none) -> Resistor_THT:R_Axial_DIN0411_L9.9mm_D3.6mm_P12.70mm_Horizontal
- RV1: footprint (none) -> Potentiometer_THT:Potentiometer_Runtron_RM-065_Vertical
- SW4, SW5, SW6: footprint (none) -> Button_Switch_THT:SW_PUSH_6mm_H5mm
Connections:
- net +5V: now also J14.4 (Pin_4)
- net A0: now also J14.12 (Pin_12)
- net A1: now also J14.11 (Pin_11)
- net A2: now also J14.10 (Pin_10)
- net A3: now also J14.9 (Pin_9)
- net A4: now also J14.8 (Pin_8)
- net A5: now also J14.7 (Pin_7)
- net A7: now also J14.5 (Pin_5)
- net D10: now also J13.13 (Pin_13)
- net D11: now also J13.14 (Pin_14)
- net D12: now also J13.15 (Pin_15)
- net D13: now also J14.15 (Pin_15)
- net D2: now also J13.5 (Pin_5)
- net D3: now also J13.6 (Pin_6)
- net D4: now also J13.7 (Pin_7)
- net D5: now also J13.8 (Pin_8)
- net D6: now also J13.9 (Pin_9)
- net D7: now also J13.10 (Pin_10)
- net D8: now also J13.11 (Pin_11)
- net D9: now also J13.12 (Pin_12)
- net Earth: now also J13.4 (Pin_4), J14.2 (Pin_2)
- net TX: now reaches A1.1 (D1/TX)
- net TX: now also J13.2 (Pin_2)
- net 3V3: now reaches A1.17 (3V3)
- net 3V3: now also J14.14 (Pin_14)
- net AREF: now reaches A1.18 (AREF)
- net AREF: now also J14.13 (Pin_13)
- net RX: now reaches A1.2 (D0/RX)
- net RX: now also J13.1 (Pin_1)
- net A6: now reaches A1.25 (A6)
- net A6: now also J14.6 (Pin_6)
- net RST: now reaches A1.28 (~RESET)
- net RST: now also A1.3 (~RESET), J13.3 (Pin_3), J14.3 (Pin_3)
- net VIN: now reaches A1.30 (VIN)
- net VIN: now also J14.1 (Pin_1)
- no-connect marks 8 -> 0
Other:
- moved on the sheet: A1, C1, C2, D7, J10, J11, J12, J4, J5, J6, J9, Q1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
