File: KiCAD_prj/ForKids/Child_bases_2/child_bases_2.sch (KiCad schematic (older format))
At the start: 39 parts

Commit message: Update Child bases 2 project
Parts:
- added D10, D11, D3, D4, D6: LED, symbol Device:LED
- added LS2: Speaker, symbol Device:Speaker
- added Q10, Q11, Q4: PN2222A, Package_TO_SOT_THT:TO-92_Inline, symbol Transistor_BJT:PN2222A
- added Q6: 2N3904*, Package_TO_SOT_THT:TO-92_Inline, symbol Transistor_BJT:2N3904
- added R10: R_PHOTO, symbol Device:R_PHOTO
- added R19, R20, R21, R22, R23, R24: R, symbol Device:R
- added R5, R8: 10K, symbol Device:R
- added R7, R9: 220, symbol Device:R
- added RV1: R_POT, symbol Device:R_POT
- added SW4: SW_DPST_x2, symbol Switch:SW_DPST_x2
- gave numbers to parts that had none: 37
Connections:
- net +9V: now also LS2.2, R19.1, R20.1, R23.1, R24.1, R5.2, R7.2, R8.2, R9.1
- net Earth: now also Q10.1 (E), Q11.1 (E), Q4.1 (E), Q6.1 (E), R10.2, SW4.2 (B), SW4.4 (B)
- net at C3.1, Q5.2 (B): now also SW2.3 (A); no longer SW2.1 (A)
- net at R12.2: now also SW2.4 (B); no longer SW2.2 (B)
- net at C1.1, Q2.2 (B): now also SW1.3 (A); no longer SW1.1 (A)
- net at R4.2: now also SW1.4 (B); no longer SW1.2 (B)
- new net: D4.2 (A), R7.1
- new net: D4.1 (K), D6.2 (A)
- new net: D6.1 (K), Q6.3 (C)
- new net: R8.1, RV1.2
- new net: Q6.2 (B), R10.1, RV1.3
- new net: D3.1 (K), LS2.1, Q4.3 (C)
- new net: D3.2 (A), R9.2
- new net: Q4.2 (B), R5.1
- new net: Q10.2 (B), R22.2, SW4.3 (A)
- new net: D10.1 (K), Q10.3 (C), R20.2, R21.2
- new net: Q11.2 (B), R21.1, SW4.1 (A)
- new net: D11.1 (K), Q11.3 (C), R22.1, R23.2
- new net: D10.2 (A), R19.2
- new net: D11.2 (A), R24.2
- no-connect marks 2 -> 5
Other:
- note added: "#1"
- note added: "#2"
- note added: "#3"
- note added: "#4"
- note added: "#5"
- note added: "#6"
- note added: "#7"
- note added: "#8. Триггер"
- note added: "#9"
- note added: "* можно заменить на 2222"
- note added: "Мультивибратор"
- note added: "Сигнализация"
- moved on the sheet: C5, C7, D8, D9, Q8, Q9, R14, R15, R16, R18

Commit message: Update Child bases 2 project
Parts:
- added C?: 100nF, symbol Device:C
- R19, R24: value R -> 470
- R20, R23: value R -> 2.2K
- R21, R22: value R -> 10K
Connections:
- net Earth: now also C?.1
- net at Q11.2 (B), R21.1, SW4.1 (A): now also C?.2
Changed lines of the file:
@@
 U 2 1 5F97CA5A
 P 5700 7150
-F 0 "SW4" H 5700 7293 50  0000 C CNN
+F 0 "SW4" H 5700 7000 50  0000 C CNN
 F 1 "SW_DPST_x2" H 5700 7293 50  0001 C CNN
 F 2 "" H 5700 7150 50  0001 C CNN
@@
 P 4300 5700
 F 0 "R20" H 4370 5746 50  0000 L CNN
-F 1 "R" H 4370 5655 50  0000 L CNN
+F 1 "2.2K" H 4370 5655 50  0000 L CNN
 F 2 "" V 4230 5700 50  0001 C CNN
 F 3 "~" H 4300 5700 50  0001 C CNN
@@
 P 6300 5750
 F 0 "R23" H 6370 5796 50  0000 L CNN
-F 1 "R" H 6370 5705 50  0000 L CNN
+F 1 "2.2K" H 6370 5705 50  0000 L CNN
 F 2 "" V 6230 5750 50  0001 C CNN
 F 3 "~" H 6300 5750 50  0001 C CNN
@@
 P 4000 5700
 F 0 "R19" H 4070 5746 50  0000 L CNN
-F 1 "R" H 4070 5655 50  0000 L CNN
+F 1 "470" H 4070 5655 50  0000 L CNN
 F 2 "" V 3930 5700 50  0001 C CNN
 F 3 "~" H 4000 5700 50  0001 C CNN
@@
 P 6600 5750
 F 0 "R24" H 6670 5796 50  0000 L CNN
-F 1 "R" H 6670 5705 50  0000 L CNN
+F 1 "470" H 6670 5705 50  0000 L CNN
 F 2 "" V 6530 5750 50  0001 C CNN
 F 3 "~" H 6600 5750 50  0001 C CNN
@@
 P 4800 6000
 F 0 "R21" V 4593 6000 50  0000 C CNN
-F 1 "R" V 4684 6000 50  0000 C CNN
+F 1 "10K" V 4684 6000 50  0000 C CNN
 F 2 "" V 4730 6000 50  0001 C CNN
 F 3 "~" H 4800 6000 50  0001 C CNN
@@
 P 5850 6000
 F 0 "R22" V 5643 6000 50  0000 C CNN
-F 1 "R" V 5734 6000 50  0000 C CNN
+F 1 "10K" V 5734 6000 50  0000 C CNN
 F 2 "" V 5780 6000 50  0001 C CNN
 F 3 "~" H 5850 6000 50  0001 C CNN
@@
 Connection ~ 4300 5350
 Wire Wire Line
-	6000 6700 5800 6700
+	6000 6700 5950 6700
 Wire Wire Line
 	4000 5350 4300 5350
@@
 	6300 6900 6300 7450
 Wire Wire Line
-	6300 7450 5700 7450
+	6300 7450 5950 7450
 Connection ~ 5700 7450
 $Comp
@@
 Wire Wire Line
 	5300 5350 6300 5350
+$Comp
+L Device:C C?
+U 1 1 5FADE233
+P 5950 7200
+F 0 "C?" H 6050 7100 50  0000 R CNN
+F 1 "100nF" H 6200 7300 50  0000 R CNN
+F 2 "" H 5988 7050 50  0001 C CNN
+F 3 "~" H 5950 7200 50  0001 C CNN
+	1    5950 7200
+	1    0    0    1
+$EndComp
+Wire Wire Line
+	5950 7350 5950 7450
+Connection ~ 5950 7450
+Wire Wire Line
+	5950 7450 5700 7450
+Wire Wire Line
+	5950 7050 5950 6700
+Connection ~ 5950 6700
+Wire Wire Line
+	5950 6700 5800 6700
 $EndSCHEMATC

Commit message: Update child bases 2 project
Parts:
- gave numbers to parts that had none: 1
Changed lines of the file:
@@
 EESchema Schematic File Version 4
-LIBS:child_bases_2-cache
 EELAYER 30 0
 EELAYER END
@@
 	5300 5350 6300 5350
 $Comp
-L Device:C C?
+L Device:C C8
 U 1 1 5FADE233
 P 5950 7200
-F 0 "C?" H 6050 7100 50  0000 R CNN
+F 0 "C8" H 6050 7100 50  0000 R CNN
 F 1 "100nF" H 6200 7300 50  0000 R CNN
 F 2 "" H 5988 7050 50  0001 C CNN
