File: KiCAD_prj/ForKids/Child_bases_2/child_bases_2.sch (KiCad schematic (older format))
At the start: 61 parts, among them Q1 PN2222A, Q10 PN2222A, Q11 PN2222A, Q2 PN2222A, Q3 PN2222A, Q4 PN2222A, Q5 PN2222A, Q6 2N3904*, Q7 PN2222A, Q8 PN2222A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

Commit message: Update chem to Child babes 1, 2 and 3
Parts:
- R20, R23: value 2.2K -> 1K
Connections:
- no-connect marks 3 -> 5
Other:
- moved on the sheet: LS1
Changed lines of the file:
@@
 U 2 1 5F982AE3
 P 6500 2350
-F 0 "SW2" H 6500 2585 50  0001 C CNN
+F 0 "SW2" H 6500 2585 50  0000 C CNN
 F 1 "SW_DPST_x2" H 6500 2493 50  0001 C CNN
 F 2 "" H 6500 2350 50  0001 C CNN
@@
 P 4300 5700
 F 0 "R20" H 4370 5746 50  0000 L CNN
-F 1 "2.2K" H 4370 5655 50  0000 L CNN
+F 1 "1K" H 4370 5655 50  0000 L CNN
 F 2 "" V 4230 5700 50  0001 C CNN
 F 3 "~" H 4300 5700 50  0001 C CNN
@@
 P 6300 5750
 F 0 "R23" H 6370 5796 50  0000 L CNN
-F 1 "2.2K" H 6370 5705 50  0000 L CNN
+F 1 "1K" H 6370 5705 50  0000 L CNN
 F 2 "" V 6230 5750 50  0001 C CNN
 F 3 "~" H 6300 5750 50  0001 C CNN
@@
 U 1 1 5FADE233
 P 5950 7200
-F 0 "C8" H 6050 7100 50  0000 R CNN
+F 0 "C8" H 6075 7100 50  0000 R CNN
 F 1 "100nF" H 6200 7300 50  0000 R CNN
 F 2 "" H 5988 7050 50  0001 C CNN
@@
 Wire Wire Line
 	4900 2350 4900 1250
-Connection ~ 3450 1250
-Wire Wire Line
-	3450 1700 3450 1250
+Wire Wire Line
+	3450 2150 3450 2050
+NoConn ~ 2200 6805
+NoConn ~ 2425 6800
+Wire Wire Line
+	2425 6800 2500 6800
 $Comp
 L Device:Speaker LS1
 U 1 1 5F978E6E
-P 3250 1700
-F 0 "LS1" H 3300 1900 50  0000 C CNN
-F 1 "Speaker" H 3250 1400 50  0000 C CNN
-F 2 "" H 3250 1500 50  0001 C CNN
-F 3 "~" H 3240 1650 50  0001 C CNN
-	1    3250 1700
+P 3250 1325
+F 0 "LS1" H 3300 1525 50  0000 C CNN
+F 1 "Speaker" H 3250 1025 50  0000 C CNN
+F 2 "" H 3250 1125 50  0001 C CNN
+F 3 "~" H 3240 1275 50  0001 C CNN
+	1    3250 1325
 	-1   0    0    -1
 $EndComp
 Wire Wire Line
-	3450 1800 3800 1800
-Wire Wire Line
-	3450 2150 3450 2050
-Wire Wire Line
-	3450 2050 3800 2050
-Wire Notes Line
-	3800 1800 3800 2050
-NoConn ~ 2200 6805
-NoConn ~ 2425 6800
-Wire Wire Line
-	2425 6800 2500 6800
+	3450 1325 3450 1250
+Connection ~ 3450 1250
+Wire Wire Line
+	3450 1425 3450 1700
+NoConn ~ 3450 1700
+NoConn ~ 3450 2050
 $EndSCHEMATC

Commit message: Update child bases 2
Parts:
- R14, R18: value 220 -> 1K
Changed lines of the file:
@@
 P 8400 4300
 F 0 "R14" H 8470 4346 50  0000 L CNN
-F 1 "220" H 8470 4255 50  0000 L CNN
+F 1 "1K" H 8470 4255 50  0000 L CNN
 F 2 "" V 8330 4300 50  0001 C CNN
 F 3 "~" H 8400 4300 50  0001 C CNN
@@
 P 10500 4300
 F 0 "R18" H 10570 4346 50  0000 L CNN
-F 1 "220" H 10570 4255 50  0000 L CNN
+F 1 "1K" H 10570 4255 50  0000 L CNN
 F 2 "" V 10430 4300 50  0001 C CNN
 F 3 "~" H 10500 4300 50  0001 C CNN

Commit message: Fix child_bases_2 projectL: remove numbers a task
Other:
- note added: "#8. Мультивибратор"
- note added: "#9. Триггер"
- note removed: "#8. Триггер"
- note removed: "#9"
- note removed: "Мультивибратор"
Changed lines of the file:
@@
 #7
 Text Notes 8450 6400 0    118  ~ 0
-#9
+#8. Мультивибратор
 Text Notes 1400 7400 0    118  ~ 0
 Сигнализация
-Text Notes 8800 6400 0    118  ~ 0
-Мультивибратор
 Wire Wire Line
 	3450 1100 3450 1250
@@
 	5350 7450 5700 7450
 Text Notes 5750 5050 0    118  ~ 0
-#8. Триггер
+#9. Триггер
 Wire Wire Line
 	4300 6000 4650 6000
