File: KiCAD_prj/ForKids/Ultraviolet/Ultraviolet.kicad_pcb (KiCad board)
At the start: 2 copper layers, 25.4 x 81.3 mm, 17 parts, among them J1 Conn_01x02_Female, SW1 SW_SPST

Commit message: Update Ultraviolet KiCad project
Routing:
- net +9V: track 124.5 -> 185.4 mm
Changed lines of the file:
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@@
     (thickness 1.6)
     (drawings 4)
-    (tracks 7)
+    (tracks 13)
     (zones 0)
     (modules 17)
@@
   )
   (setup
-    (last_trace_width 1)
+    (last_trace_width 0.25)
     (user_trace_width 1)
     (trace_clearance 0.2)
@@
   (segment (start 142.24 85.09) (end 142.24 31.75) (width 1) (layer B.Cu) (net 1))
   (segment (start 132.08 31.75) (end 142.24 31.75) (width 1) (layer B.Cu) (net 1))
+  (segment (start 132.08 40.64) (end 142.24 40.64) (width 1) (layer B.Cu) (net 1))
+  (segment (start 132.08 49.53) (end 142.24 49.53) (width 1) (layer B.Cu) (net 1))
+  (segment (start 132.08 58.42) (end 142.24 58.42) (width 1) (layer B.Cu) (net 1))
+  (segment (start 132.08 67.31) (end 142.24 67.31) (width 1) (layer B.Cu) (net 1))
+  (segment (start 132.08 76.2) (end 142.24 76.2) (width 1) (layer B.Cu) (net 1))
+  (segment (start 132.08 85.09) (end 142.24 85.09) (width 1) (layer B.Cu) (net 1))
   (segment (start 144.943 101.31) (end 144.9705 101.2825) (width 1) (layer B.Cu) (net 3))
   (segment (start 132.08 101.31) (end 144.943 101.31) (width 1) (layer B.Cu) (net 3))
