File: KiCAD_prj/ForKids/Child_bases_3/Child_bases_3.sch (KiCad schematic (older format))
At the start: 8 parts, among them M1 Motor_DC, SW1 SW_DPST_x2, SW2 SW_DPST_x2

Commit message: Update chem to Child babes 1, 2 and 3
Parts:
- M2: renamed from M?; value Motor_DC -> Motor_DC: 3V
- RV1: renamed from RV?; value R_POT -> 10K
- gave numbers to parts that had none: 3
Connections:
- net Earth: now also SW1.3 (A), SW2.3 (A); no longer SW1.4 (B), SW2.4 (B)
- net at M1.1 (+), SW2.2 (B): now also SW2.4 (B); no longer SW2.3 (A)
- net at M1.2 (-), SW1.2 (B): now also SW1.4 (B); no longer SW1.3 (A)
Other:
- note added: "#2"
- moved on the sheet: D1, M2, Q1, R1, RV1
Changed lines of the file:
@@
 F 3 "~" H 1750 3150 50  0001 C CNN
 	2    1750 3150
-	0    -1   1    0
+	0    -1   -1   0
 $EndComp
 $Comp
@@
 F 3 "~" H 2900 3150 50  0001 C CNN
 	2    2900 3150
-	0    1    1    0
+	0    1    -1   0
 $EndComp
 Wire Wire Line
@@
 Motor bridge
 $Comp
-L Transistor_BJT:PN2222A Q?
+L Transistor_BJT:PN2222A Q1
 U 1 1 5FA4F10B
-P 4800 2900
-F 0 "Q?" H 4990 2946 50  0000 L CNN
-F 1 "PN2222A" H 4990 2855 50  0000 L CNN
-F 2 "Package_TO_SOT_THT:TO-92_Inline" H 5000 2825 50  0001 L CIN
-F 3 "https://www.onsemi.com/pub/Collateral/PN2222-D.PDF" H 4800 2900 50  0001 L CNN
-	1    4800 2900
-	1    0    0    -1
-$EndComp
-$Comp
-L Device:R R?
+P 4750 2850
+F 0 "Q1" H 4940 2896 50  0000 L CNN
+F 1 "PN2222A" H 4940 2805 50  0000 L CNN
+F 2 "Package_TO_SOT_THT:TO-92_Inline" H 4950 2775 50  0001 L CIN
+F 3 "https://www.onsemi.com/pub/Collateral/PN2222-D.PDF" H 4750 2850 50  0001 L CNN
+	1    4750 2850
+	1    0    0    -1
+$EndComp
+$Comp
+L Device:R R1
 U 1 1 5FA4F474
-P 4350 3200
-F 0 "R?" H 4280 3154 50  0000 R CNN
-F 1 "1K" H 4280 3245 50  0000 R CNN
-F 2 "" V 4280 3200 50  0001 C CNN
-F 3 "~" H 4350 3200 50  0001 C CNN
-	1    4350 3200
+P 4300 3150
+F 0 "R1" H 4230 3104 50  0000 R CNN
+F 1 "1K" H 4230 3195 50  0000 R CNN
+F 2 "" V 4230 3150 50  0001 C CNN
+F 3 "~" H 4300 3150 50  0001 C CNN
+	1    4300 3150
 	-1   0    0    1
 $EndComp
 $Comp
-L Motor:Motor_DC M?
+L Motor:Motor_DC M2
 U 1 1 5FA4FB55
-P 4900 2150
-F 0 "M?" H 5100 2100 50  0000 L CNN
-F 1 "Motor_DC" H 5100 2000 50  0000 L CNN
-F 2 "" H 4900 2060 50  0001 C CNN
-F 3 "~" H 4900 2060 50  0001 C CNN
-	1    4900 2150
-	1    0    0    -1
-$EndComp
-$Comp
-L Diode:1N4001 D?
+P 4850 2100
+F 0 "M2" H 5050 2100 50  0000 L CNN
+F 1 "Motor_DC: 3V" H 5050 2025 50  0000 L CNN
+F 2 "" H 4850 2010 50  0001 C CNN
+F 3 "~" H 4850 2010 50  0001 C CNN
+	1    4850 2100
+	1    0    0    -1
+$EndComp
+$Comp
+L Diode:1N4001 D1
 U 1 1 5FA53298
-P 4550 2200
-F 0 "D?" V 4504 2280 50  0000 L CNN
-F 1 "1N4001" V 4650 1850 50  0000 L CNN
-F 2 "Diode_THT:D_DO-41_SOD81_P10.16mm_Horizontal" H 4550 2025 50  0001 C CNN
-F 3 "http://www.vishay.com/docs/88503/1n4001.pdf" H 4550 2200 50  0001 C CNN
-	1    4550 2200
+P 4500 2150
+F 0 "D1" V 4400 2000 50  0000 L CNN
+F 1 "1N4001" V 4500 1825 50  0000 L CNN
+F 2 "Diode_THT:D_DO-41_SOD81_P10.16mm_Horizontal" H 4500 1975 50  0001 C CNN
+F 3 "http://www.vishay.com/docs/88503/1n4001.pdf" H 4500 2150 50  0001 C CNN
+	1    4500 2150
 	0    1    1    0
 $EndComp
 Wire Wire Line
-	4550 2050 4550 1900
-Wire Wire Line
-	4550 1900 4900 1900
-Wire Wire Line
-	4550 2350 4550 2550
-Wire Wire Line
-	4550 2550 4900 2550
-Wire Wire Line
-	4900 2550 4900 2450
-Wire Wire Line
-	4900 2700 4900 2550
-Connection ~ 4900 2550
-$Comp
-L power:+5V #PWR?
+	4500 2000 4500 1850
+Wire Wire Line
+	4500 1850 4850 1850
+Wire Wire Line
+	4500 2300 4500 2500
+Wire Wire Line
+	4500 2500 4850 2500
+Wire Wire Line
+	4850 2500 4850 2400
+Wire Wire Line
+	4850 2650 4850 2500
+Connection ~ 4850 2500
+$Comp
+L power:+5V #PWR02
 U 1 1 5FA5666B
-P 4900 1700
-F 0 "#PWR?" H 4900 1550 50  0001 C CNN
-F 1 "+5V" H 4915 1873 50  0000 C CNN
-F 2 "" H 4900 1700 50  0001 C CNN
-F 3 "" H 4900 1700 50  0001 C CNN
-	1    4900 1700
-	1    0    0    -1
-$EndComp
-Wire Wire Line
-	4900 1700 4900 1900
-Connection ~ 4900 1900
-Wire Wire Line
-	4900 1900 4900 1950
-$Comp
-L power:Earth #PWR?
+P 4850 1650
+F 0 "#PWR02" H 4850 1500 50  0001 C CNN
+F 1 "+5V" H 4865 1823 50  0000 C CNN
+F 2 "" H 4850 1650 50  0001 C CNN
+F 3 "" H 4850 1650 50  0001 C CNN
+	1    4850 1650
+	1    0    0    -1
+$EndComp
+Wire Wire Line
+	4850 1650 4850 1850
+Connection ~ 4850 1850
+Wire Wire Line
+	4850 1850 4850 1900
+$Comp
+L power:Earth #PWR03
 U 1 1 5FA58272
-P 4900 3700
-F 0 "#PWR?" H 4900 3450 50  0001 C CNN
-F 1 "Earth" H 4900 3550 50  0001 C CNN
-F 2 "" H 4900 3700 50  0001 C CNN
-F 3 "~" H 4900 3700 50  0001 C CNN
-	1    4900 3700
-	1    0    0    -1
-$EndComp
-Wire Wire Line
-	4600 2900 4350 2900
-Wire Wire Line
-	4900 3100 4900 3500
-Wire Wire Line
-	4350 3350 4350 3500
-Wire Wire Line
-	4350 3500 4900 3500
-Connection ~ 4900 3500
-Wire Wire Line
-	4900 3500 4900 3700
-$Comp
-L Device:R_POT RV?
+P 4850 3650
+F 0 "#PWR03" H 4850 3400 50  0001 C CNN
+F 1 "Earth" H 4850 3500 50  0001 C CNN
+F 2 "" H 4850 3650 50  0001 C CNN
+F 3 "~" H 4850 3650 50  0001 C CNN
+	1    4850 3650
+	1    0    0    -1
+$EndComp
+Wire Wire Line
+	4550 2850 4300 2850
+Wire Wire Line
+	4850 3050 4850 3450
+Wire Wire Line
+	4300 3300 4300 3450
+Wire Wire Line
+	4300 3450 4850 3450
+Connection ~ 4850 3450
+Wire Wire Line
+	4850 3450 4850 3650
+$Comp
+L Device:R_POT RV1
 U 1 1 5FA5FDD0
-P 4350 2650
-F 0 "RV?" H 4280 2696 50  0000 R CNN
-F 1 "R_POT" H 4280 2605 50  0000 R CNN
-F 2 "" H 4350 2650 50  0001 C CNN
-F 3 "~" H 4350 2650 50  0001 C CNN
-	1    4350 2650
+P 4300 2600
+F 0 "RV1" H 4230 2646 50  0000 R CNN
+F 1 "10K" H 4230 2555 50  0000 R CNN
+F 2 "" H 4300 2600 50  0001 C CNN
+F 3 "~" H 4300 2600 50  0001 C CNN
+	1    4300 2600
 	-1   0    0    -1
 $EndComp
 Wire Wire Line
-	4350 2800 4350 2900
-Connection ~ 4350 2900
-Wire Wire Line
-	4350 2900 4350 3050
-Wire Wire Line
-	4200 2650 3950 2650
-$Comp
-L power:+5V #PWR?
+	4300 2750 4300 2850
+Connection ~ 4300 2850
+Wire Wire Line
+	4300 2850 4300 3000
+Wire Wire Line
+	4150 2600 3900 2600
+$Comp
+L power:+5V #PWR01
 U 1 1 5FA62BBC
-P 3950 1700
-F 0 "#PWR?" H 3950 1550 50  0001 C CNN
-F 1 "+5V" H 3965 1873 50  0000 C CNN
-F 2 "" H 3950 1700 50  0001 C CNN
-F 3 "" H 3950 1700 50  0001 C CNN
-	1    3950 1700
-	1    0    0    -1
-$EndComp
-Wire Wire Line
-	3950 1700 3950 2650
+P 3900 1650
+F 0 "#PWR01" H 3900 1500 50  0001 C CNN
+F 1 "+5V" H 3915 1823 50  0000 C CNN
+F 2 "" H 3900 1650 50  0001 C CNN
+F 3 "" H 3900 1650 50  0001 C CNN
+	1    3900 1650
+	1    0    0    -1
+$EndComp
+Wire Wire Line
+	3900 1650 3900 2600
+Text Notes 4250 1225 0    118  ~ 0
+#2
 $EndSCHEMATC
